Commit message: Expand run_scenarios to compare OSQP and Crocoddyl

File: bauzil_stairs.urdf (robot description, URDF)
Before this commit: robot bauzil_stairs.urdf, 1 links, 0 joints
Links:
- link baseLink: geometry collision mesh filename=bauzil_stairs.stl scale=1.3 1.3 0.4; visual mesh filename=bauzil_stairs.stl scale=1.3 1.3 0.4
